File: top_controller/top_controller.kicad_pcb (KiCad board)
At the start: 2 copper layers, 117 parts, among them J1 OUT1, J10 USB_C_Receptacle_USB2.0, J11 SWD, J12 UART, J13 BOOT0, J14 BOOT1, J2 OUT2, J3 OUT3, J4 OUT4, J5 OUT5, J6 OUT6, J7 OUT7, J8 OUT8, J9 PIN, SW1 RESET, U1 STM32F103C8Tx, U2 LT3045xMSE, U3 AD5754BREZ, U4 AD5754BREZ, U5 REF192, U6 EPM78V2, U7 REF192, Y1 8MHz

Commit message: Finished all the traces (except connecting two grounds and testpoints on SPI)
Parts:
- moved TP16 425.7 mm to (74.0, 141.9)
- moved TP17 425.7 mm to (74.0, 146.9)
- moved TP19 425.7 mm to (79.0, 126.8)
- moved TP20 425.7 mm to (79.0, 131.8)
- moved TP21 425.7 mm to (79.0, 136.8)
- moved TP18 422.5 mm to (79.4, 119.9)
- moved R1 9.26 mm to (208.3, 48.2)
- moved R30 9.25 mm to (217.5, 49.3)
- moved J14 3.75 mm to (214.8, 52.8)
- moved J13 3.75 mm to (211.0, 52.8)
- moved R22 1.70 mm to (232.2, 35.0), turned to 180 degrees
- moved R3 1.55 mm to (223.2, 67.8)
- moved Y1 1.55 mm to (223.8, 73.3)
Routing:
- net VDDA: track 64.6 -> 198.0 mm, vias 0 -> 6
- net /SPI_CLK: track 128.3 -> 226.3 mm, vias 2 -> 4
- net /SPI_D2D: track 18.0 -> 114.9 mm, vias 2 -> 4
- net /NLDAC: track 127.4 -> 223.3 mm, vias 2 -> 4
- net /SPI_NSS: track 128.2 -> 223.4 mm
- net /NCLR: track 126.2 -> 220.9 mm, vias 2 -> 4
- net /SPI_MISO: track 114.6 -> 177.4 mm, vias 2 -> 6
- net +3V3: track 219.9 -> 282.0 mm, vias 5 -> 13
- net /BOOT0: track 3.69 -> 25.3 mm, vias 1 -> 2
- net /BOOT1: track 0.00 -> 20.2 mm, vias 0 -> 2
- net /PIN_VCC: track 43.0 -> 54.8 mm, vias 0 -> 1
- net /USB_VBUS: track 59.5 -> 70.8 mm
- net GNDA: track 66.6 -> 77.1 mm, vias 14 -> 19
- net /LED_CH2: track 84.9 -> 86.2 mm
- net /LED_CH1: track 61.0 -> 62.1 mm
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- added copper zone on B.Cu, net GND
- added copper zone on F.Cu, net GND
- added copper zone on B.Cu, net GNDA

Commit message: Finished tracing - still some errors present
Parts:
- moved TP16 115.7 mm to (169.8, 77.1), turned to -90 degrees
- moved TP17 115.3 mm to (165.7, 77.1), turned to -90 degrees
- moved TP19 96.3 mm to (161.6, 77.1), turned to -90 degrees
- moved TP20 92.3 mm to (153.4, 77.1), turned to -90 degrees
- moved TP21 92.2 mm to (149.3, 77.1), turned to -90 degrees
- moved TP18 89.1 mm to (157.5, 77.1), turned to -90 degrees
Connections:
- C12 pad 2: GNDA -> GND
- C13 pad 2: GNDA -> GND
- C16 pad 2: GNDA -> GND
- C17 pad 2: GNDA -> GND
- C18 pad 2: GNDA -> GND
- C20 pad 2: GNDA -> GND
- C21 pad 2: GNDA -> GND
- C22 pad 2: GNDA -> GND
- C23 pad 2: GNDA -> GND
- C24 pad 2: GNDA -> GND
- C25 pad 2: GNDA -> GND
- C26 pad 2: GNDA -> GND
- C27 pad 2: GNDA -> GND
- C28 pad 2: GNDA -> GND
- C29 pad 2: GNDA -> GND
- C30 pad 2: GNDA -> GND
- D13 pad 1: GNDA -> GND
- D14 pad 1: GNDA -> GND
- J1 pad 2: GNDA -> GND
- J2 pad 2: GNDA -> GND
- J3 pad 2: GNDA -> GND
- J4 pad 2: GNDA -> GND
- J5 pad 2: GNDA -> GND
- J6 pad 2: GNDA -> GND
- J7 pad 2: GNDA -> GND
- J8 pad 2: GNDA -> GND
- J9 pad 2: GNDA -> GND
- R13 pad 2: GNDA -> GND
- R14 pad 2: GNDA -> GND
- R15 pad 2: GNDA -> GND
- R16 pad 2: GNDA -> GND
- R17 pad 2: GNDA -> GND
- R18 pad 2: GNDA -> GND
- R19 pad 2: GNDA -> GND
- R20 pad 2: GNDA -> GND
- TP4 pad 1: GNDA -> GND
- U3 pad 1: GNDA -> GND
- U3 pad 15: GNDA -> GND
- U3 pad 18: GNDA -> GND
- U3 pad 19: GNDA -> GND
- U3 pad 20: GNDA -> GND
- U3 pad 21: GNDA -> GND
- U3 pad 25: GNDA -> GND
- U4 pad 1: GNDA -> GND
- U4 pad 15: GNDA -> GND
- U4 pad 18: GNDA -> GND
- U4 pad 19: GNDA -> GND
- U4 pad 20: GNDA -> GND
- U4 pad 21: GNDA -> GND
- U4 pad 25: GNDA -> GND
- U5 pad 4: GNDA -> GND
- U6 pad 2: GNDA -> GND
- U7 pad 4: GNDA -> GND
Routing:
- net GND: track 81.2 -> 158.3 mm, vias 17 -> 36
- net GNDA: track 77.1 -> 0.00 mm, vias 19 -> 0
- net /SPI_MISO: track 177.4 -> 182.9 mm
- net /SPI_CLK: track 226.3 -> 231.8 mm
- net /SPI_NSS: track 223.4 -> 228.9 mm
- net /NLDAC: track 223.3 -> 228.7 mm
- net /NCLR: track 220.9 -> 226.2 mm
- net /SPI_MOSI: track 128.6 -> 133.9 mm
- net /REF_2V5_1: track 23.7 -> 28.1 mm
- removed copper zone on B.Cu, net GNDA
- removed copper zone on F.Cu, net GNDA
